File: hdmi-cec/pcb/claudobip-hdmi-cec.sch (EAGLE design)
At the start: 26 parts, among them IC1 LD117AV33, Q1 16mhz, SW1 PUSH_BUTTON_SWITCH, T1 2N3904, T2 2N3904, U1 ATMEGA328P-AU, X2 MINI-USB_5P

Commit message: [HDMI-CEC] Use a vertical footprint for the LD117AV33 regulator
Parts:
- IC1: value LD117AV33 -> LD117AV33-VERTICAL; device v-reg:LD117AV33 -> regulator:LD117AV33-VERTICAL
